Commit message: Add files via upload

File: src/jetbot/urdf/jetbot.urdf (robot description, URDF)
Before this commit: robot jetbot.zip, 7 links, 6 joints
Links:
- removed link rueda_derecha_link
- removed link rueda_izquierda_link
- added link camera_link, mass 0.0018; collision mesh filename=package://jetbot/meshes/camera_link.STL; visual mesh filename=package://jetbot/meshes/camera_link.STL
- added link derecha_abajo_link, mass 0.0871203991688674; collision mesh filename=package://jetbot/meshes/derecha_abajo_link.STL; visual mesh filename=package://jetbot/meshes/derecha_abajo_link.STL
- added link derecha_arriba_link, mass 0.008712; collision mesh filename=package://jetbot/meshes/derecha_arriba_link.STL; visual mesh filename=package://jetbot/meshes/derecha_arriba_link.STL
- added link izquierda_abajo_link, mass 0.0087120399168867; collision mesh filename=package://jetbot/meshes/izquierda_abajo_link.STL; visual mesh filename=package://jetbot/meshes/izquierda_abajo_link.STL
- added link izquierda_arriba_link, mass 0.0087120399168867; collision mesh filename=package://jetbot/meshes/izquierda_arriba_link.STL; visual mesh filename=package://jetbot/meshes/izquierda_arriba_link.STL
- link cabeza_link: mass 0.127124344939099 -> 0.0127
- link cuello_link: mass 0.1152446218733567 -> 0.0152
- link subir_link: mass 0.1273663857179312 -> 0.0273
Joints:
- removed joint rueda_derecha_joint
- removed joint rueda_izquierda_joint
- added joint camera_joint: type fixed, parent cabeza_link, child camera_link, origin xyz=0.030723 -0.0098391 0.032 rpy=0.33531 1.5708 0, axis 0 0 0
- added joint derecha_abajo_joint: type continuous, parent base_link, child derecha_abajo_link, origin xyz=-0.061638 -0.060627 -0.024684 rpy=1.5708 0 3.1416, axis 0 0 1, limit effort=100 velocity=100
- added joint derecha_arriba_joint: type continuous, parent base_link, child derecha_arriba_link, origin xyz=0.048098 -0.061627 -0.024956 rpy=-1.5708 -0.22688 0, axis 0 0 1, limit effort=100 velocity=100
- added joint izquierda_abajo_joint: type continuous, parent base_link, child izquierda_abajo_link, origin xyz=-0.061638 0.060786 -0.024684 rpy=-1.5708 0 3.1416, axis 0 0 1, limit effort=100 velocity=100
- added joint izquierda_arriba_joint: type continuous, parent base_link, child izquierda_arriba_link, origin xyz=0.04845 0.060786 -0.024684 rpy=-1.5708 0 3.1416, axis 0 0 1, limit effort=100 velocity=100
- joint cabeza_joint: limit lower=-0.7 upper=0.35 effort=100 velocity=100 -> lower=-1.6 upper=0.5 effort=100 velocity=100; origin xyz=0.00027896605587166 0.0322637933061906 0.0102106923628102 rpy=-1.5707963267949 -0.471467109281761 0 -> xyz=0.00027 0.032264 0.010211 rpy=-1.5708 0 -3.1416
- joint camera_optical_joint: origin xyz=0.00027896605587166 -0.0322637933061906 0.0102106923628102 rpy=0 0 0 -> xyz=1 1 1 rpy=0.3 0.3 0.3; parent cabeza_link -> camera_link
- joint cuello_joint: origin xyz=-0.0192210339441284 -0.000736206693809111 0.0493487604025714 rpy=0 0 3.14159265358979 -> xyz=0.0192 0.0007 0.0493 rpy=0 0 0
- joint subir_joint: origin xyz=0.075406 7.7147E-05 0.083651 rpy=0 0 0 -> xyz=0.075406 7.7147E-05 0.083651 rpy=0 0 3.1416
